File: led_daughterboard/led_daughterboard.kicad_sch (KiCad schematic)
At the start: 12 parts, among them J1 STM32 Black Pill L, J2 STM32 Black Pill R, J3 Barrel_Jack, J4 INMP441_1, J5 INMP441_2, J6 LED_Out, SW1 SW_Push, U1 SN74LV1T34DBV

Commit message: Start the messy tracing
Connections:
- net +5V: now also J1.18 (Pin_18); no longer J2.1 (Pin_1)
Changed lines of the file:
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@@
-	(wire
-		(pts
-			(xy 154.94 57.15) (xy 151.13 57.15)
-		)
-		(stroke
-			(width 0)
-			(type default)
-		)
-	)
 	(wire
 		(pts
@@
 	(symbol
 		(lib_id "power:+5V")
-		(at 154.94 57.15 270)
+		(at 124.46 100.33 90)
 		(mirror x)
 		(unit 1)
@@
 		(fields_autoplaced yes)
 		(property "Reference" "#PWR06"
-			(at 151.13 57.15 0)
+			(at 128.27 100.33 0)
 			(effects
 				(font
@@
 		)
 		(property "Value" "+5V"
-			(at 158.75 57.1499 90)
-			(effects
-				(font
-					(size 1.27 1.27)
-				)
-				(justify left)
+			(at 123.19 97.79 90)
+			(effects
+				(font
+					(size 1.27 1.27)
+				)
 			)
 		)
 		(property "Footprint" ""
-			(at 154.94 57.15 0)
+			(at 124.46 100.33 0)
 			(effects
 				(font
@@
 		)
 		(property "Datasheet" ""
-			(at 154.94 57.15 0)
+			(at 124.46 100.33 0)
 			(effects
 				(font
@@
 		)
 		(property "Description" "Power symbol creates a global label with name \"+5V\""
-			(at 154.94 57.15 0)
-			(effects
-				(font
+			(at 124.46 100.33 0)
+			(effects
+				(font
